Commit message: FEAT: Add camera on gazebo

File: arduinobot_description/urdf/arduinobot.urdf.xacro (robot description, xacro)
@@ -4,4 +4,5 @@
     <xacro:property name="effort" value="30.0" />
     <xacro:property name="velocity" value="10.0" />
+    <xacro:arg name="is_ignition" default="true"/>
     <xacro:macro name="default_inertial" params="mass">
         <inertial>
@@ -158,7 +159,7 @@
         <limit lower="0.0" upper="${PI/2}" effort="${effort}" velocity="${velocity}"/>
     </joint>
-    <!-- <link name="rgb_camera">
-        <visual>
-            <origin rpy="-1.57 0.0 -1.57" xyz="-0.1 0.125 0.135"/>
+    <link name="rgb_camera">
+        <visual>
+            <origin rpy="-1.57 0 -1.57" xyz="-0.1 0.125 0.15"/>
             <geometry>
                 <mesh filename="package://arduinobot_description/meshes/pi_camera.STL" scale="0.01 0.01 0.01"/>
@@ -166,9 +167,12 @@
         </visual>
         <collision>
-            <origin rpy="-1.57 0.0 -1.57" xyz="-0.1 0.125 0.135"/>
+            <origin rpy="-1.57 0 -1.57" xyz="-0.1 0.125 0.15"/>
             <geometry>
                 <mesh filename="package://arduinobot_description/meshes/pi_camera.STL" scale="0.01 0.01 0.01"/>
             </geometry>
         </collision>
+        <inertial>
+            <mass value="0.001"/>
+        </inertial>
     </link>
     <joint name="rgb_camera_joint" type="fixed">
@@ -176,4 +180,49 @@
         <child link="rgb_camera"/>
         <origin rpy="0 -0.5 1.57" xyz="0 0.45 0.2"/>
-    </joint> -->
+    </joint>
+    <gazebo reference="rgb_camera">
+        <sensor name="camera" type="camera">
+            <always_on>true</always_on>
+            <update_rate>30.0</update_rate>
+            <visualize>true</visualize>
+            <topic>/image_raw</topic>
+            <gz_frame_id>/rgb_camera</gz_frame_id>
+            <camera name="camera">
+            <horizontal_fov>1.21126</horizontal_fov>
+            <image>
+                <width>2304</width>
+                <height>1296</height>
+                <format>R8G8B8</format>
+            </image>
+            <distortion>
+                <k1>0.0</k1>
+                <k2>0.0</k2>
+                <k3>0.0</k3>
+                <p1>0.0</p1>
+                <p2>0.0</p2>
+                <center>0.5 0.5</center>
+            </distortion>
+            </camera>
+        </sensor>
+    </gazebo>
+    <gazebo>
+    <!-- ROS 2 Humble -->
+    <xacro:if value="$(arg is_ignition)">
+        <!-- <plugin filename="ign_ros2_control-system" name="ign_ros2_control::IgnitionROS2ControlPlugin">
+        <parameters>$(find arduinobot_controller)/config/arduinobot_controllers.yaml</parameters>
+        </plugin> -->
+        <plugin filename="ignition-gazebo-sensors-system" name="ignition::gazebo::systems::Sensors">
+        <render_engine>ogre2</render_engine>
+        </plugin>
+    </xacro:if>
+    <!-- ROS 2 Iron or above -->
+    <xacro:unless value="$(arg is_ignition)">
+        <!-- <plugin filename="gz_ros2_control-system" name="gz_ros2_control::GazeboSimROS2ControlPlugin">
+        <parameters>$(find arduinobot_controller)/config/arduinobot_controllers.yaml</parameters>
+        </plugin> -->
+        <plugin filename="gz-sim-sensors-system" name="gz::sim::systems::Sensors">
+        <render_engine>ogre2</render_engine>
+        </plugin>
+    </xacro:unless>
+    </gazebo>
 </robot>

Commit message: FIX: Using corret names

File: arduinobot_description/urdf/arduinobot.urdf.xacro (robot description, xacro)
@@ -1,10 +1,15 @@
 <?xml version="1.0"?>
 <robot xmlns:xacro="http://www.ros.org/wiki/xacro" name="arduinobot">
+    <!-- Start GZ or Ignition depending on ROS 2 Version -->
+    <xacro:arg name="is_ignition" default="true"/>
+    <!-- Load Simulated or Real Hardware Interfaces -->
+    <xacro:arg name="is_sim" default="true"/>
+    <!-- Include Gazebo Parameters -->
+    <xacro:include filename="$(find arduinobot_description)/urdf/arduinobot_gazebo.xacro" />
+    <!-- Include ros2_control Plugins -->
+    <xacro:include filename="$(find arduinobot_description)/urdf/arduinobot_ros2_control.xacro" />
     <xacro:property name="PI" value="3.14159" />
     <xacro:property name="effort" value="30.0" />
     <xacro:property name="velocity" value="10.0" />
-    <xacro:arg name="is_ignition" default="true"/>
-    <xacro:include filename="$(find arduinobot_description)/urdf/arduinobot_gazebo.xacro" />
-    <xacro:include filename="$(find arduinobot_description)/urdf/arduinobot_ros2_control.xacro" />
     <xacro:macro name="default_inertial" params="mass">
         <inertial>

File: arduinobot_description/urdf/arduinobot_gazebo.xacro (robot description, xacro)
@@ -1,48 +1,49 @@
 <?xml version="1.0"?>
 <robot xmlns:xacro="http://www.ros.org/wiki/xacro" name="arduinobot">
-     <gazebo>
+  <!-- ROS 2 Control -->
+  <gazebo>
     <!-- ROS 2 Humble -->
     <xacro:if value="$(arg is_ignition)">
-        <plugin filename="ign_ros2_control-system" name="ign_ros2_control::IgnitionROS2ControlPlugin">
+      <plugin filename="ign_ros2_control-system" name="ign_ros2_control::IgnitionROS2ControlPlugin">
         <parameters>$(find arduinobot_controller)/config/arduinobot_controllers.yaml</parameters>
-        </plugin>
-        <plugin filename="ignition-gazebo-sensors-system" name="ignition::gazebo::systems::Sensors">
+      </plugin>
+      <plugin filename="ignition-gazebo-sensors-system" name="ignition::gazebo::systems::Sensors">
         <render_engine>ogre2</render_engine>
-        </plugin>
+      </plugin>
     </xacro:if>
     <!-- ROS 2 Iron or above -->
     <xacro:unless value="$(arg is_ignition)">
-        <plugin filename="gz_ros2_control-system" name="gz_ros2_control::GazeboSimROS2ControlPlugin">
+      <plugin filename="gz_ros2_control-system" name="gz_ros2_control::GazeboSimROS2ControlPlugin">
         <parameters>$(find arduinobot_controller)/config/arduinobot_controllers.yaml</parameters>
-        </plugin>
-        <plugin filename="gz-sim-sensors-system" name="gz::sim::systems::Sensors">
+      </plugin>
+      <plugin filename="gz-sim-sensors-system" name="gz::sim::systems::Sensors">
         <render_engine>ogre2</render_engine>
-        </plugin>
+      </plugin>
     </xacro:unless>
-    </gazebo>
-    <gazebo reference="rgb_camera">
-        <sensor name="camera" type="camera">
-            <always_on>true</always_on>
-            <update_rate>30.0</update_rate>
-            <visualize>true</visualize>
-            <topic>/image_raw</topic>
-            <gz_frame_id>/rgb_camera</gz_frame_id>
-            <camera name="camera">
-            <horizontal_fov>1.21126</horizontal_fov>
-            <image>
-                <width>2304</width>
-                <height>1296</height>
-                <format>R8G8B8</format>
-            </image>
-            <distortion>
-                <k1>0.0</k1>
-                <k2>0.0</k2>
-                <k3>0.0</k3>
-                <p1>0.0</p1>
-                <p2>0.0</p2>
-                <center>0.5 0.5</center>
-            </distortion>
-            </camera>
-        </sensor>
-    </gazebo>
+  </gazebo>
+  <gazebo reference="rgb_camera">
+    <sensor name="camera" type="camera">
+        <always_on>true</always_on>
+        <update_rate>30.0</update_rate>
+        <visualize>true</visualize>
+        <topic>/image_raw</topic>
+        <gz_frame_id>/rgb_camera</gz_frame_id>
+        <camera name="camera">
+          <horizontal_fov>1.21126</horizontal_fov>
+          <image>
+            <width>2304</width>
+            <height>1296</height>
+            <format>R8G8B8</format>
+          </image>
+          <distortion>
+            <k1>0.0</k1>
+            <k2>0.0</k2>
+            <k3>0.0</k3>
+            <p1>0.0</p1>
+            <p2>0.0</p2>
+            <center>0.5 0.5</center>
+          </distortion>
+        </camera>
+    </sensor>
+</gazebo>
 </robot>

File: arduinobot_description/urdf/arduinobot_ros2_control.xacro (robot description, xacro)
@@ -1,20 +1,36 @@
 <?xml version="1.0"?>
 <robot xmlns:xacro="http://www.ros.org/wiki/xacro" name="arduinobot">
-    <xacro:property name="PI" value="3.14159" />
-    <ros2_control type="system" name="RobotSystem">
-        <xacro:if value="$(arg is_ignition)">
-             <hardware>
-                <plugin>ign_ros2_control/IgnitionSystem</plugin>
-            </hardware>
+    <ros2_control name="RobotSystem" type="system">
+        <xacro:property name="PI" value="3.14159265359" />
+        <!-- ros2_control Gazebo -->
+        <xacro:if value="$(arg is_sim)">
+            <!-- ROS 2 Humble -->
+            <xacro:if value="$(arg is_ignition)">
+                <hardware>
+                    <plugin>ign_ros2_control/IgnitionSystem</plugin>
+                </hardware>
+            </xacro:if>
+            <!-- ROS 2 Iron or above -->
+            <xacro:unless value="$(arg is_ignition)">
+                <hardware>
+                    <plugin>gz_ros2_control/GazeboSimSystem</plugin>
+                </hardware>
+            </xacro:unless>
+            <joint name="joint_5">
+                <param name="mimic">joint_4</param>
+                <param name="multiplier">-1</param>
+            </joint>
         </xacro:if>
-        <xacro:unless value="$(arg is_ignition)">
+        <!-- ros2_control Real Robot -->
+        <xacro:unless value="$(arg is_sim)">
             <hardware>
-                <plugin>gz_ros2_control/GazeboSimSystem</plugin>
+                <plugin>arduinobot_controller/ArduinobotInterface</plugin>
+                <param name="port">/dev/ttyACM0</param>
             </hardware>
         </xacro:unless>
         <joint name="joint_1">
             <command_interface name="position">
-                <param name="min">-${PI/2}</param>
-                <param name="max">${PI/2}</param>
+            <param name="min">-${PI / 2}</param>
+            <param name="max">${PI / 2}</param>
             </command_interface>
             <state_interface name="position"/>
@@ -22,6 +38,6 @@
         <joint name="joint_2">
             <command_interface name="position">
-                <param name="min">-${PI/2}</param>
-                <param name="max">${PI/2}</param>
+            <param name="min">-${PI / 2}</param>
+            <param name="max">${PI / 2}</param>
             </command_interface>
             <state_interface name="position"/>
@@ -29,6 +45,6 @@
         <joint name="joint_3">
             <command_interface name="position">
-                <param name="min">-${PI/2}</param>
-                <param name="max">${PI/2}</param>
+            <param name="min">-${PI / 2}</param>
+            <param name="max">${PI / 2}</param>
             </command_interface>
             <state_interface name="position"/>
@@ -36,13 +52,9 @@
         <joint name="joint_4">
             <command_interface name="position">
-                <param name="min">-${PI/2}</param>
-                <param name="max">0.0</param>
+            <param name="min">-${PI / 2}</param>
+            <param name="max">0.0</param>
             </command_interface>
             <state_interface name="position"/>
         </joint>
-        <joint name="joint_5">
-                <param name="mimic">joint_4</param>
-                <param name="multiplier">-1</param>
-        </joint>
     </ros2_control>
 </robot>

Commit message: REFACTOR: Add color on robot

File: arduinobot_description/urdf/arduinobot.urdf.xacro (robot description, xacro)
@@ -28,4 +28,7 @@
                 <mesh filename="package://arduinobot_description/meshes/basement.STL" scale="0.01 0.01 0.01"/>
             </geometry>
+            <material name="blue">
+                <color rgba="0.1 0.1 0.8 1.0"/>
+            </material>
         </visual>
         <collision>
@@ -48,4 +51,7 @@
                 <mesh filename="package://arduinobot_description/meshes/base_plate.STL" scale="0.01 0.01 0.01"/>
             </geometry>
+            <material name="grey">
+                <color rgba="0.5 0.5 0.5 1.0"/>
+            </material>
         </visual>
         <collision>
@@ -70,4 +76,7 @@
                 <mesh filename="package://arduinobot_description/meshes/forward_drive_arm.STL" scale="0.01 0.01 0.01"/>
             </geometry>
+            <material name="grey">
+                <color rgba="0.5 0.5 0.5 1.0"/>
+            </material>
         </visual>
     </link>
@@ -86,4 +95,7 @@
                 <mesh filename="package://arduinobot_description/meshes/horizontal_arm.STL" scale="0.01 0.01 0.01"/>
             </geometry>
+            <material name="grey">
+                <color rgba="0.5 0.5 0.5 1.0"/>
+            </material>
         </visual>
         <collision>
@@ -108,4 +120,7 @@
                 <mesh filename="package://arduinobot_description/meshes/claw_support.STL" scale="0.01 0.01 0.01"/>
             </geometry>
+            <material name="grey">
+                <color rgba="0.5 0.5 0.5 1.0"/>
+            </material>
         </visual>
         <collision>
@@ -128,4 +143,7 @@
                 <mesh filename="package://arduinobot_description/meshes/right_finger.STL" scale="0.01 0.01 0.01"/>
             </geometry>
+            <material name="blue">
+                <color rgba="0.1 0.1 0.8 1.0"/>
+            </material>
         </visual>
         <collision>
@@ -143,4 +161,7 @@
                 <mesh filename="package://arduinobot_description/meshes/left_finger.STL" scale="0.01 0.01 0.01"/>
             </geometry>
+            <material name="blue">
+                <color rgba="0.1 0.1 0.8 1.0"/>
+            </material>
         </visual>
         <collision>
@@ -172,4 +193,7 @@
                 <mesh filename="package://arduinobot_description/meshes/pi_camera.STL" scale="0.01 0.01 0.01"/>
             </geometry>
+            <material name="purple">
+                <color rgba="0.8 0.1 0.8 1.0"/>
+            </material>
         </visual>
         <collision>
@@ -188,3 +212,28 @@
         <origin rpy="0 -0.5 1.57" xyz="0 0.45 0.2"/>
     </joint>
+    <gazebo reference="rgb_camera">
+        <sensor name="rgb_camera" type="camera">
+            <always_on>true</always_on>
+            <update_rate>30.0</update_rate>
+            <visualize>true</visualize>
+            <topic>/image_raw</topic>
+            <gz_frame_id>/rgb_camera</gz_frame_id>
+            <camera name="camera">
+            <horizontal_fov>1.21126</horizontal_fov>
+            <image>
+                <width>2304</width>
+                <height>1296</height>
+                <format>R8G8B8</format>
+            </image>
+            <distortion>
+                <k1>0.0</k1>
+                <k2>0.0</k2>
+                <k3>0.0</k3>
+                <p1>0.0</p1>
+                <p2>0.0</p2>
+                <center>0.5 0.5</center>
+            </distortion>
+            </camera>
+        </sensor>
+    </gazebo>
 </robot>

File: arduinobot_description/urdf/arduinobot_gazebo.xacro (robot description, xacro)
@@ -22,28 +22,3 @@
     </xacro:unless>
   </gazebo>
-  <gazebo reference="rgb_camera">
-    <sensor name="camera" type="camera">
-        <always_on>true</always_on>
-        <update_rate>30.0</update_rate>
-        <visualize>true</visualize>
-        <topic>/image_raw</topic>
-        <gz_frame_id>/rgb_camera</gz_frame_id>
-        <camera name="camera">
-          <horizontal_fov>1.21126</horizontal_fov>
-          <image>
-            <width>2304</width>
-            <height>1296</height>
-            <format>R8G8B8</format>
-          </image>
-          <distortion>
-            <k1>0.0</k1>
-            <k2>0.0</k2>
-            <k3>0.0</k3>
-            <p1>0.0</p1>
-            <p2>0.0</p2>
-            <center>0.5 0.5</center>
-          </distortion>
-        </camera>
-    </sensor>
-</gazebo>
 </robot>

Commit message: REFACTOR: Remove inertial to show camera

File: arduinobot_description/urdf/arduinobot.urdf.xacro (robot description, xacro)
@@ -189,5 +189,5 @@
     <link name="rgb_camera">
         <visual>
-            <origin rpy="-1.57 0 -1.57" xyz="-0.1 0.125 0.15"/>
+            <origin rpy="-1.57 0 -1.57" xyz="-0.07 0.13 0.15"/>
             <geometry>
                 <mesh filename="package://arduinobot_description/meshes/pi_camera.STL" scale="0.01 0.01 0.01"/>
@@ -198,12 +198,9 @@
         </visual>
         <collision>
-            <origin rpy="-1.57 0 -1.57" xyz="-0.1 0.125 0.15"/>
+            <origin rpy="-1.57 0 -1.57" xyz="-0.1 0.13 0.15"/>
             <geometry>
                 <mesh filename="package://arduinobot_description/meshes/pi_camera.STL" scale="0.01 0.01 0.01"/>
             </geometry>
         </collision>
-        <inertial>
-            <mass value="0.001"/>
-        </inertial>
     </link>
     <joint name="rgb_camera_joint" type="fixed">
